File: PCB/SpinningLight/SpinningLight.kicad_pcb (KiCad board)
At the start: 2 copper layers, 106.7 x 78.7 mm, 30 parts, among them J0 Power, J1 Neopixel, J10 3V3, J11 5VCC, J2 Temperature Sensor, J3 OLED, J4 Reset, J5 Reserve IO23 5VCC, J6 Reserve IO25 5VCC, J7 Reserve IO09 3V3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

Commit message: improved the pcb by enlarging the holes for the level shifter
previously, the holes of the level shifter were too small making it effectively a pressfit. It has been improved here.
Routing:
- net 3V3: track 194.3 -> 190.0 mm, vias 1 -> 3
Changed lines of the file:
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@@
     (fp_rect (start -6.35 -16.51) (end 8.89 -3.81)
       (stroke (width 0.1) (type default)) (fill none) (layer "F.SilkS"))
-    (pad "1" thru_hole circle (at -5.08 -5.08) (size 1.524 1.524) (drill 0.762) (layers "*.Cu" "*.Mask" "Eco2.User")
+    (pad "1" thru_hole circle (at -5.08 -5.08) (size 2 2) (drill 1) (layers "*.Cu" "*.Mask" "Eco2.User")
       (net 26 "Net-(U1-IO_05{slash}D8)") (pinfunction "LV1") (pintype "bidirectional"))
-    (pad "2" thru_hole circle (at -2.54 -5.08) (size 1.524 1.524) (drill 0.762) (layers "*.Cu" "*.Mask")
+    (pad "2" thru_hole circle (at -2.54 -5.08) (size 2 2) (drill 1) (layers "*.Cu" "*.Mask")
       (net 34 "Net-(U1-IO_17{slash}D3)") (pinfunction "LV2") (pintype "bidirectional"))
-    (pad "3" thru_hole circle (at 0 -5.08) (size 1.524 1.524) (drill 0.762) (layers "*.Cu" "*.Mask")
+    (pad "3" thru_hole circle (at 0 -5.08) (size 2 2) (drill 1) (layers "*.Cu" "*.Mask")
       (net 5 "3V3") (pinfunction "LV") (pintype "bidirectional"))
-    (pad "4" thru_hole circle (at 2.54 -5.08) (size 1.524 1.524) (drill 0.762) (layers "*.Cu" "*.Mask")
+    (pad "4" thru_hole circle (at 2.54 -5.08) (size 2 2) (drill 1) (layers "*.Cu" "*.Mask")
       (net 3 "GND") (pinfunction "GND") (pintype "bidirectional"))
-    (pad "5" thru_hole circle (at 5.08 -5.08) (size 1.524 1.524) (drill 0.762) (layers "*.Cu" "*.Mask")
+    (pad "5" thru_hole circle (at 5.08 -5.08) (size 2 2) (drill 1) (layers "*.Cu" "*.Mask")
       (net 24 "Net-(U1-IO_23{slash}D7)") (pinfunction "LV3") (pintype "bidirectional"))
-    (pad "6" thru_hole circle (at 7.62 -5.08) (size 1.524 1.524) (drill 0.762) (layers "*.Cu" "*.Mask")
+    (pad "6" thru_hole circle (at 7.62 -5.08) (size 2 2) (drill 1) (layers "*.Cu" "*.Mask")
       (net 32 "Net-(U1-IO_25)") (pinfunction "LV4") (pintype "bidirectional"))
-    (pad "7" thru_hole circle (at -5.08 -15.24) (size 1.524 1.524) (drill 0.762) (layers "*.Cu" "*.Mask")
+    (pad "7" thru_hole circle (at -5.08 -15.24) (size 2 2) (drill 1) (layers "*.Cu" "*.Mask")
       (net 2 "Net-(J1-Pin_2)") (pinfunction "HV1") (pintype "bidirectional"))
-    (pad "8" thru_hole circle (at -2.54 -15.24) (size 1.524 1.524) (drill 0.762) (layers "*.Cu" "*.Mask")
+    (pad "8" thru_hole circle (at -2.54 -15.24) (size 2 2) (drill 1) (layers "*.Cu" "*.Mask")
       (net 4 "Net-(J2-Pin_2)") (pinfunction "HV2") (pintype "bidirectional"))
-    (pad "9" thru_hole circle (at 0 -15.24) (size 1.524 1.524) (drill 0.762) (layers "*.Cu" "*.Mask")
+    (pad "9" thru_hole circle (at 0 -15.24) (size 2 2) (drill 1) (layers "*.Cu" "*.Mask")
       (net 1 "5VCC") (pinfunction "HV") (pintype "bidirectional"))
-    (pad "10" thru_hole circle (at 2.54 -15.24) (size 1.524 1.524) (drill 0.762) (layers "*.Cu" "*.Mask")
+    (pad "10" thru_hole circle (at 2.54 -15.24) (size 2 2) (drill 1) (layers "*.Cu" "*.Mask")
       (net 3 "GND") (pinfunction "GND") (pintype "bidirectional"))
-    (pad "11" thru_hole circle (at 5.08 -15.24) (size 1.524 1.524) (drill 0.762) (layers "*.Cu" "*.Mask")
+    (pad "11" thru_hole circle (at 5.08 -15.24) (size 2 2) (drill 1) (layers "*.Cu" "*.Mask")
       (net 8 "Net-(J5-Pin_2)") (pinfunction "HV3") (pintype "bidirectional"))
-    (pad "12" thru_hole circle (at 7.62 -15.24) (size 1.524 1.524) (drill 0.762) (layers "*.Cu" "*.Mask")
+    (pad "12" thru_hole circle (at 7.62 -15.24) (size 2 2) (drill 1) (layers "*.Cu" "*.Mask")
       (net 9 "Net-(J6-Pin_2)") (pinfunction "HV4") (pintype "bidirectional"))
   )
@@
   (segment (start 157.48 83.82) (end 138.525 64.865) (width 0.25) (layer "B.Cu") (net 4))
   (segment (start 129.13 97.79) (end 109.22 97.79) (width 0.25) (layer "F.Cu") (net 5))
-  (segment (start 161.473 83.369749) (end 161.473 92.527) (width 0.25) (layer "F.Cu") (net 5))
   (segment (start 198.12 109.22) (end 196.605 110.735) (width 0.25) (layer "F.Cu") (net 5))
   (segment (start 190.679569 115.57) (end 167.64 115.57) (width 0.25) (layer "F.Cu") (net 5))
   (segment (start 177.8 64.135) (end 175.895 64.135) (width 0.25) (layer "F.Cu") (net 5))
   (segment (start 160.02 111.77) (end 161.28 113.03) (width 0.25) (layer "F.Cu") (net 5))
+  (segment (start 171.214081 82.733) (end 171.214081 84.055919) (width 0.25) (layer "F.Cu") (net 5))
   (segment (start 109.22 99.06) (end 109.22 96.52) (width 0.25) (layer "F.Cu") (net 5))
-  (segment (start 161.473 92.527) (end 160.02 93.98) (width 0.25) (layer "F.Cu") (net 5))
+  (segment (start 161.473 92.527) (end 161.29 92.71) (width 0.25) (layer "F.Cu") (net 5))
   (segment (start 175.895 64.135) (end 173.99 66.04) (width 0.25) (layer "F.Cu") (net 5))
   (segment (start 196.605 110.735) (end 195.155431 110.735) (width 0.25) (layer "F.Cu") (net 5))
@@
   (segment (start 135.52 104.18) (end 129.13 97.79) (width 0.25) (layer "F.Cu") (net 5))
   (segment (start 181.255 67.59) (end 177.8 64.135) (width 0.25) (layer "F.Cu") (net 5))
-  (segment (start 162.109749 82.733) (end 161.473 83.369749) (width 0.25) (layer "F.Cu") (net 5))
   (segment (start 161.28 113.03) (end 160.105 114.205) (width 0.25) (layer "F.Cu") (net 5))
   (segment (start 138.195 114.205) (end 135.52 116.88) (width 0.25) (layer "F.Cu") (net 5))
+  (segment (start 161.29 92.71) (end 160.02 93.98) (width 0.25) (layer "F.Cu") (net 5))
   (segment (start 109.22 101.6) (end 109.22 99.06) (width 0.25) (layer "F.Cu") (net 5))
   (segment (start 194.065 111.825431) (end 194.065 112.184569) (width 0.25) (layer "F.Cu") (net 5))
   (segment (start 194.065 112.184569) (end 190.679569 115.57) (width 0.25) (layer "F.Cu") (net 5))
-  (segment (start 171.214081 82.733) (end 162.109749 82.733) (width 0.25) (layer "F.Cu") (net 5))
   (segment (start 195.155431 110.735) (end 194.065 111.825431) (width 0.25) (layer "F.Cu") (net 5))
   (segment (start 135.52 116.88) (end 135.52 110.29) (width 0.25) (layer "F.Cu") (net 5))
@@
   (segment (start 160.105 114.205) (end 138.195 114.205) (width 0.25) (layer "F.Cu") (net 5))
   (segment (start 135.52 110.29) (end 135.52 104.18) (width 0.25) (layer "F.Cu") (net 5))
+  (segment (start 171.214081 84.055919) (end 170.18 85.09) (width 0.25) (layer "F.Cu") (net 5))
   (via (at 167.64 115.57) (size 0.8) (drill 0.4) (layers "F.Cu" "B.Cu") (net 5))
+  (via (at 161.29 92.71) (size 0.8) (drill 0.4) (layers "F.Cu" "B.Cu") (net 5))
+  (via (at 170.18 85.09) (size 0.8) (drill 0.4) (layers "F.Cu" "B.Cu") (net 5))
   (segment (start 167.64 115.57) (end 163.82 115.57) (width 0.25) (layer "B.Cu") (net 5))
+  (segment (start 169.576167 85.09) (end 161.956167 92.71) (width 0.25) (layer "B.Cu") (net 5))
+  (segment (start 161.956167 92.71) (end 161.29 92.71) (width 0.25) (layer "B.Cu") (net 5))
   (segment (start 163.82 115.57) (end 161.28 113.03) (width 0.25) (layer "B.Cu") (net 5))
+  (segment (start 170.18 85.09) (end 169.576167 85.09) (width 0.25) (layer "B.Cu") (net 5))
   (segment (start 165.1 110.49) (end 185.42 90.17) (width 0.25) (layer "F.Cu") (net 6))
   (segment (start 185.42 90.17) (end 185.42 86.36) (width 0.25) (layer "F.Cu") (net 6))
@@
   (segment (start 182.455431 85.335) (end 181.365 86.425431) (width 0.25) (layer "B.Cu") (net 32))
   (segment (start 181.365 86.425431) (end 181.365 86.784569) (width 0.25) (layer "B.Cu") (net 32))
-  (segment (start 186.445 83.395431) (end 185.844569 82.795) (width 0.25) (layer "B.Cu") (net 34))
-  (segment (start 160.287251 92.71) (end 158.75 92.71) (width 0.25) (layer "B.Cu") (net 34))
   (segment (start 187.535431 85.335) (end 186.445 84.244569) (width 0.25) (layer "B.Cu") (net 34))
-  (segment (start 185.844569 82.795) (end 170.202251 82.795) (width 0.25) (layer "B.Cu") (net 34))
-  (segment (start 190.5 86.36) (end 189.475 85.335) (width 0.25) (layer "B.Cu") (net 34))
+  (segment (start 185.844569 82.795) (end 171.021125 82.795) (width 0.25) (layer "B.Cu") (net 34))
   (segment (start 189.475 85.335) (end 187.535431 85.335) (width 0.25) (layer "B.Cu") (net 34))
   (segment (start 186.445 84.244569) (end 186.445 83.395431) (width 0.25) (layer "B.Cu") (net 34))
-  (segment (start 170.202251 82.795) (end 160.287251 92.71) (width 0.25) (layer "B.Cu") (net 34))
-  (segment (start 158.75 92.71) (end 157.48 93.98) (width 0.25) (layer "B.Cu") (net 34))
+  (segment (start 190.5 86.36) (end 189.475 85.335) (width 0.25) (layer "B.Cu") (net 34))
+  (segment (start 163.646125 90.17) (end 161.29 90.17) (width 0.25) (layer "B.Cu") (net 34))
+  (segment (start 171.021125 82.795) (end 163.646125 90.17) (width 0.25) (layer "B.Cu") (net 34))
+  (segment (start 186.445 83.395431) (end 185.844569 82.795) (width 0.25) (layer "B.Cu") (net 34))
+  (segment (start 161.29 90.17) (end 157.48 93.98) (width 0.25) (layer "B.Cu") (net 34))
 )
